File: hardware/relayConnector.kicad_sch (KiCad schematic)
At the start: 1 part, among them J401 Screw_Terminal_01x03

Commit message: added manual and picture
Changed lines of the file:
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@@
 	(paper "A4")
 	(bus_entry
-		(at 97.79 82.55)
+		(at 116.84 82.55)
 		(size 2.54 -2.54)
 		(stroke
@@
 	)
 	(bus_entry
-		(at 97.79 87.63)
+		(at 116.84 87.63)
 		(size 2.54 -2.54)
-		(stroke
-			(width 0)
-			(type default)
-		)
-	)
-	(wire
-		(pts
-			(xy 83.82 87.63) (xy 97.79 87.63)
-		)
 		(stroke
 			(width 0)
@@
 	(bus
 		(pts
-			(xy 100.33 77.47) (xy 100.33 80.01)
+			(xy 119.38 77.47) (xy 119.38 80.01)
 		)
 		(stroke
@@
 	(wire
 		(pts
-			(xy 83.82 82.55) (xy 97.79 82.55)
+			(xy 83.82 82.55) (xy 116.84 82.55)
 		)
 		(stroke
@@
 		)
 	)
-	(bus
+	(wire
 		(pts
-			(xy 100.33 80.01) (xy 100.33 85.09)
+			(xy 83.82 87.63) (xy 116.84 87.63)
 		)
 		(stroke
@@
 	(bus
 		(pts
-			(xy 102.87 77.47) (xy 100.33 77.47)
+			(xy 119.38 80.01) (xy 119.38 85.09)
+		)
+		(stroke
+			(width 0)
+			(type default)
+		)
+	)
+	(bus
+		(pts
+			(xy 121.92 77.47) (xy 119.38 77.47)
 		)
 		(stroke
@@
 	)
 	(label "pin1"
-		(at 92.71 82.55 0)
-		(fields_autoplaced yes)
+		(at 111.76 82.55 0)
 		(effects
 			(font
@@
 	)
 	(label "pin2"
-		(at 92.71 87.63 0)
-		(fields_autoplaced yes)
+		(at 111.76 87.63 0)
 		(effects
 			(font
@@
 	(hierarchical_label "{relays}"
 		(shape input)
-		(at 102.87 77.47 0)
-		(fields_autoplaced yes)
+		(at 121.92 77.47 0)
 		(effects
 			(font
